File: ESP32-A1S-Tayloe-kicad/ESP32-A1S-Tayloe-kicad.sch (KiCad schematic (older format))
At the start: 11 parts

Commit message: gg
Parts:
- added Q1, Q2: 2N3904, Package_TO_SOT_THT:TO-92_Inline, symbol Transistor_BJT:2N3904
- added R1, R2: Resistor, symbol esp32-a1s-rescue:Resistor-Xenir
- added SW1: SW_DIP_x01, symbol Switch:SW_DIP_x01
- added U2: USB_to_Serial, symbol esp32-a1s-rescue:USB_to_Serial-Xenir
- gave numbers to parts that had none: 11
Connections:
- net labels added: DTR, EN, IO0, RTS, RX0, TX0
- net labels removed: +3.3V, SERIALRX, SERIALTX
- wire segments 42 -> 57
Other:
- moved on the sheet: C1, C2, C3, C4, D1, J1, R3, R4, SW2, U1, U3

Commit message: gg
Parts:
- added C5, C6: 22uF, symbol xenir:Cap_Polarized
Connections:
- net OUTL: now also C6.1; no longer R4.2
- net OUTR: now also C5.1; no longer R3.2
- new net: C5.2, R3.2
- new net: C6.2, R4.2
Other:
- moved on the sheet: C1, C2, J1, R3, R4
Changed lines of the file:
@@
 L xenir:Audio_Jack J1
 U 1 1 62B4F5DF
-P 3200 5800
-F 0 "J1" H 3183 5831 50  0000 C CNN
-F 1 "Audio_Jack" H 3183 5740 50  0000 C CNN
-F 2 "" H 3200 5800 50  0001 C CNN
-F 3 "" H 3200 5800 50  0001 C CNN
-	1    3200 5800
+P 2750 5800
+F 0 "J1" H 2733 5831 50  0000 C CNN
+F 1 "Audio_Jack" H 2733 5740 50  0000 C CNN
+F 2 "" H 2750 5800 50  0001 C CNN
+F 3 "" H 2750 5800 50  0001 C CNN
+	1    2750 5800
 	1    0    0    1
 $EndComp
@@
 L xenir:Capacitor C1
 U 1 1 62B508AF
-P 3950 5400
-F 0 "C1" H 3950 5550 28  0000 C CNN
-F 1 ".1uF" H 4050 5450 28  0000 C CNN
-F 2 "" H 3950 5250 50  0001 C CNN
-F 3 "" H 3950 5250 50  0001 C CNN
-	1    3950 5400
+P 3500 5400
+F 0 "C1" H 3500 5550 28  0000 C CNN
+F 1 ".1uF" H 3600 5450 28  0000 C CNN
+F 2 "" H 3500 5250 50  0001 C CNN
+F 3 "" H 3500 5250 50  0001 C CNN
+	1    3500 5400
 	0    1    1    0
 $EndComp
@@
 L xenir:Capacitor C2
 U 1 1 62B50F6B
-P 4300 5650
-F 0 "C2" H 4300 5800 28  0000 C CNN
-F 1 ".1uF" H 4400 5700 28  0000 C CNN
-F 2 "" H 4300 5500 50  0001 C CNN
-F 3 "" H 4300 5500 50  0001 C CNN
-	1    4300 5650
+P 3850 5650
+F 0 "C2" H 3850 5800 28  0000 C CNN
+F 1 ".1uF" H 3950 5700 28  0000 C CNN
+F 2 "" H 3850 5500 50  0001 C CNN
+F 3 "" H 3850 5500 50  0001 C CNN
+	1    3850 5650
 	0    1    1    0
 $EndComp
@@
 L xenir:Resistor R3
 U 1 1 62B531E9
-P 4550 5250
-F 0 "R3" H 4550 5404 28  0000 C CNN
-F 1 "330" H 4550 5347 28  0000 C CNN
-F 2 "" H 4550 5150 50  0001 C CNN
-F 3 "" H 4550 5150 50  0001 C CNN
-	1    4550 5250
+P 4100 5250
+F 0 "R3" H 4100 5404 28  0000 C CNN
+F 1 "330" H 4100 5347 28  0000 C CNN
+F 2 "" H 4100 5150 50  0001 C CNN
+F 3 "" H 4100 5150 50  0001 C CNN
+	1    4100 5250
 	1    0    0    -1
 $EndComp
@@
 L xenir:Resistor R4
 U 1 1 62B53AF7
-P 4550 5500
-F 0 "R4" H 4550 5654 28  0000 C CNN
-F 1 "330" H 4550 5597 28  0000 C CNN
-F 2 "" H 4550 5400 50  0001 C CNN
-F 3 "" H 4550 5400 50  0001 C CNN
-	1    4550 5500
+P 4100 5500
+F 0 "R4" H 4100 5654 28  0000 C CNN
+F 1 "330" H 4100 5597 28  0000 C CNN
+F 2 "" H 4100 5400 50  0001 C CNN
+F 3 "" H 4100 5400 50  0001 C CNN
+	1    4100 5500
 	1    0    0    -1
 $EndComp
@@
 L power:GND #PWR04
 U 1 1 62B556EE
-P 3950 5550
-F 0 "#PWR04" H 3950 5300 50  0001 C CNN
-F 1 "GND" H 3955 5377 50  0000 C CNN
-F 2 "" H 3950 5550 50  0001 C CNN
-F 3 "" H 3950 5550 50  0001 C CNN
-	1    3950 5550
+P 3500 5550
+F 0 "#PWR04" H 3500 5300 50  0001 C CNN
+F 1 "GND" H 3505 5377 50  0000 C CNN
+F 2 "" H 3500 5550 50  0001 C CNN
+F 3 "" H 3500 5550 50  0001 C CNN
+	1    3500 5550
 	1    0    0    -1
 $EndComp
@@
 L power:GND #PWR06
 U 1 1 62B55B43
-P 4300 5800
-F 0 "#PWR06" H 4300 5550 50  0001 C CNN
-F 1 "GND" H 4305 5627 50  0000 C CNN
-F 2 "" H 4300 5800 50  0001 C CNN
-F 3 "" H 4300 5800 50  0001 C CNN
-	1    4300 5800
-	1    0    0    -1
-$EndComp
-Wire Wire Line
-	4850 5250 4750 5250
-Wire Wire Line
-	4850 5500 4750 5500
-Wire Wire Line
-	4350 5500 4300 5500
-Wire Wire Line
-	4350 5250 3950 5250
-Wire Wire Line
-	3400 5350 3650 5350
-Wire Wire Line
-	3650 5350 3650 5250
-Wire Wire Line
-	3650 5250 3950 5250
-Connection ~ 3950 5250
-Wire Wire Line
-	3400 5450 3650 5450
-Wire Wire Line
-	3650 5450 3650 5500
-Wire Wire Line
-	3650 5500 4300 5500
-Connection ~ 4300 5500
+P 3850 5800
+F 0 "#PWR06" H 3850 5550 50  0001 C CNN
+F 1 "GND" H 3855 5627 50  0000 C CNN
+F 2 "" H 3850 5800 50  0001 C CNN
+F 3 "" H 3850 5800 50  0001 C CNN
+	1    3850 5800
+	1    0    0    -1
+$EndComp
+Wire Wire Line
+	3900 5500 3850 5500
+Wire Wire Line
+	3900 5250 3500 5250
+Wire Wire Line
+	2950 5350 3200 5350
+Wire Wire Line
+	3200 5350 3200 5250
+Wire Wire Line
+	3200 5250 3500 5250
+Connection ~ 3500 5250
+Wire Wire Line
+	2950 5450 3200 5450
+Wire Wire Line
+	3200 5450 3200 5500
+Wire Wire Line
+	3200 5500 3850 5500
+Connection ~ 3850 5500
 $Comp
 L power:GND #PWR03
 U 1 1 62B5D275
-P 3400 5650
-F 0 "#PWR03" H 3400 5400 50  0001 C CNN
-F 1 "GND" H 3405 5477 50  0000 C CNN
-F 2 "" H 3400 5650 50  0001 C CNN
-F 3 "" H 3400 5650 50  0001 C CNN
-	1    3400 5650
+P 2950 5650
+F 0 "#PWR03" H 2950 5400 50  0001 C CNN
+F 1 "GND" H 2955 5477 50  0000 C CNN
+F 2 "" H 2950 5650 50  0001 C CNN
+F 3 "" H 2950 5650 50  0001 C CNN
+	1    2950 5650
 	1    0    0    -1
 $EndComp
@@
 Wire Wire Line
 	6250 5500 6800 5500
+$Comp
+L xenir:Cap_Polarized C5
+U 1 1 62CE938D
+P 4550 5350
+F 0 "C5" H 4550 5046 28  0000 C CNN
+F 1 "22uF" H 4550 5103 28  0000 C CNN
+F 2 "" H 4550 5400 50  0001 C CNN
+F 3 "" H 4550 5400 50  0001 C CNN
+	1    4550 5350
+	-1   0    0    1
+$EndComp
+$Comp
+L xenir:Cap_Polarized C6
+U 1 1 62CEA988
+P 4550 5600
+F 0 "C6" H 4550 5650 28  0000 C CNN
+F 1 "22uF" H 4550 5700 28  0000 C CNN
+F 2 "" H 4550 5650 50  0001 C CNN
+F 3 "" H 4550 5650 50  0001 C CNN
+	1    4550 5600
+	-1   0    0    1
+$EndComp
+Wire Wire Line
+	4700 5250 4850 5250
+Wire Wire Line
+	4700 5500 4850 5500
+Wire Wire Line
+	4400 5250 4300 5250
+Wire Wire Line
+	4400 5500 4300 5500
 $EndSCHEMATC
